Commit message: 6/19 SDF 파일 수정 - 조인트 결합 문제 수정

File: agv_description/urdf/agv.urdf.xacro (robot description, xacro)
@@ -5,5 +5,5 @@
     <parent link="base_footprint" />
     <child link="base_link" />
-    <origin xyz="0 0 0" rpy="0 0 0" />
+    <origin xyz="0 0 0.1" rpy="0 0 0" />
   </joint>
   <link name="base_link">
@@ -22,7 +22,131 @@
       <origin xyz="0 0 0" rpy="0 0 0" />
       <geometry>
-        <box size="2 2 2"/>
+        <mesh filename="package://agv_description/meshes/BODY.stl" />
       </geometry>
     </collision>
   </link>
+  <joint name="mast_joint" type="fixed">
+    <parent link="base_link" />
+    <child link="mast" />
+    <origin xyz="0 0.631 1.875" rpy="0 0 0" />
+  </joint>
+  <link name="mast">
+    <inertial>
+      <mass value="590.628"/>
+      <inertia ixx="1122.228" ixy="-0.195" ixz="1.265" iyy="1071.349" iyz="-243.104" izz="135.921"/>
+    </inertial>
+    <visual>
+      <origin xyz="0 0 0" rpy="0 0 0" />
+      <geometry>
+        <mesh filename="package://agv_description/meshes/MAST_RE.stl" />
+      </geometry>
+      <material name="dark_grey" />
+    </visual>
+    <collision>
+      <origin xyz="0 0 0" rpy="0 0 0" />
+      <geometry>
+        <mesh filename="package://agv_description/meshes/MAST_RE.stl" />
+      </geometry>
+    </collision>
+  </link>
+  <joint name="front_wheel_l_joint" type="continuous">
+    <parent link="base_link" />
+    <child link="front_wheel_l" />
+    <origin xyz="-0.451 0.86 0.035" rpy="0 0 -1.571" />
+    <axis xyz="0 1 0"/>
+  </joint>
+  <link name="front_wheel_l">
+    <inertial>
+      <mass value="16.096"/>
+      <inertia ixx="0.066" ixy="0.0" ixz="0.0" iyy="0.104" iyz="0.0" izz="0.066"/>
+    </inertial>
+    <visual>
+      <origin xyz="0 0 0" rpy="0 0 0" />
+      <geometry>
+        <mesh filename="package://agv_description/meshes/FRONT_WHEEL_RE2.stl"/>
+      </geometry>
+      <material name="green" />
+    </visual>
+    <collision>
+      <origin xyz="0 0 0" rpy="0 0 0" />
+      <geometry>
+        <mesh filename="package://agv_description/meshes/FRONT_WHEEL_RE2.stl"/>
+      </geometry>
+    </collision>
+  </link>
+  <joint name="front_wheel_r_joint" type="continuous">
+    <parent link="base_link" />
+    <child link="front_wheel_r" />
+    <origin xyz="0.451 0.86 0.035" rpy="0 0 1.571" />
+    <axis xyz="0 1 0"/>
+  </joint>
+  <link name="front_wheel_r">
+    <inertial>
+      <mass value="16.096"/>
+      <inertia ixx="0.066" ixy="0.0" ixz="0.0" iyy="0.104" iyz="0.0" izz="0.066"/>
+    </inertial>
+    <visual>
+      <origin xyz="0 0 0" rpy="0 0 0" />
+      <geometry>
+        <mesh filename="package://agv_description/meshes/FRONT_WHEEL_RE2.stl"/>
+      </geometry>
+      <material name="green" />
+    </visual>
+    <collision>
+      <origin xyz="0 0 0" rpy="0 0 0" />
+      <geometry>
+        <mesh filename="package://agv_description/meshes/FRONT_WHEEL_RE2.stl"/>
+      </geometry>
+    </collision>
+  </link>
+  <!-- <joint name="steering_joint" type="continuous">
+    <parent link="base_link" />
+    <child link="steering_part" />
+    <origin xyz="-0.0456 -0.212 0.375" rpy="0 0 0" />
+    <axis xyz="0 0 1"/>
+  </joint>
+  <link name="steering_part">
+    <inertial>
+      <mass value="85.056"/>
+      <inertia ixx="2.77" ixy="0.0" ixz="0.12" iyy="2.81" iyz="-0.11" izz="0.9"/>
+    </inertial>
+    <visual>
+      <origin xyz="0 0 0" rpy="0 0 0" />
+      <geometry>
+        <mesh filename="package://agv_description/meshes/STEERING_PART_RE2.stl"/>
+      </geometry>
+      <material name="white" />
+    </visual>
+    <collision>
+      <origin xyz="0 0 0" rpy="0 0 0" />
+      <geometry>
+        <mesh filename="package://agv_description/meshes/STEERING_PART_RE2.stl"/>
+      </geometry>
+    </collision>
+  </link>
+  <joint name="drive_wheel_joint" type="continuous">
+    <parent link="steering_part" />
+    <child link="drive_wheel" />
+    <origin xyz="0.063 0.012 -0.285" rpy="0 0 0" />
+    <axis xyz="1 0 0"/>
+  </joint>
+  <link name="drive_wheel">
+    <inertial>
+      <mass value="21.755"/>
+      <inertia ixx="0.265" ixy="0.0" ixz="0.0" iyy="0.166" iyz="0.0" izz="0.166"/>
+    </inertial>
+    <visual>
+      <origin xyz="0 0 0" rpy="0 0 0" />
+      <geometry>
+        <mesh filename="package://agv_description/meshes/DRIVE_WHEEL_RE2.stl"/>
+      </geometry>
+      <material name="blue" />
+    </visual>
+    <collision>
+      <origin xyz="0 0 0" rpy="0 0 0" />
+      <geometry>
+        <mesh filename="package://agv_description/meshes/DRIVE_WHEEL_RE2.stl"/>
+      </geometry>
+    </collision>
+  </link> -->
 </robot>

File: agv_description/urdf/agv1.urdf .xacro (robot description, xacro)
@@ -100,14 +100,38 @@
     </collision>
   </link>
-  <joint name="steering_joint" type="continuous">
+  <joint name="steering_motor_joint" type="continuous">
     <parent link="base_link" />
+    <child link="steering_mortor" />
+    <origin xyz="0.185 -0.2 0.466" rpy="0 0 0" />
+    <axis xyz="0 0 1"/>
+  </joint>
+  <link name="steering_motor">
+    <inertial>
+      <mass value="10"/>
+      <inertia ixx="0.462" ixy="0.0" ixz="-0.002" iyy="0.462" iyz="0.0" izz="0.033"/>
+    </inertial>
+    <visual>
+      <origin xyz="0 0 0" rpy="0 0 0" />
+      <geometry>
+        <mesh filename="package://agv_description/meshes/STEERING_MOTOR.stl" scale="0.001 0.001 0.001"/>
+      </geometry>
+      <material name="white" />
+    </visual>
+    <collision>
+      <origin xyz="0 0 0" rpy="0 0 3.14" />
+      <geometry>
+        <mesh filename="package://agv_description/meshes/STEERING_MOTOR.stl" scale="0.001 0.001 0.001"/>
+      </geometry>
+    </collision>
+  </link>
+  <joint name="steering_joint" type="fixed">
+    <parent link="steering_motor" />
     <child link="steering_part" />
     <origin xyz="0.0456 -0.212 0.375" rpy="0 0 0" />
-    <axis xyz="0 0 1"/>
   </joint>
   <link name="steering_part">
     <inertial>
-      <mass value="85.197"/>
-      <inertia ixx="2.8" ixy="0.0" ixz="0.11" iyy="2.84" iyz="-0.11" izz="0.93"/>
+      <mass value="85.056"/>
+      <inertia ixx="2.77" ixy="0.0" ixz="0.12" iyy="2.81" iyz="-0.11" izz="0.9"/>
     </inertial>
     <visual>
@@ -134,5 +158,5 @@
     <inertial>
       <mass value="21.755"/>
-      <inertia ixx="2.03" ixy="0.02" ixz="-0.42" iyy="2.03" iyz="-0.07" izz="0.27"/>
+      <inertia ixx="0.265" ixy="0.0" ixz="0.0" iyy="0.166" iyz="0.0" izz="0.166"/>
     </inertial>
     <visual>
