Commit message: 패키지 명 변경 description > sim

File: agv_sim/urdf/agv.urdf (robot description, URDF)
Before this commit: robot agv1, 5 links, 4 joints
Links:
- added link drive_wheel, mass 21.755; collision mesh filename=package://agv_sim/meshes/DRIVE_WHEEL_RE2.stl; visual mesh filename=package://agv_sim/meshes/DRIVE_WHEEL_RE2.stl
- added link steering_part, mass 85.197; collision mesh filename=package://agv_sim/meshes/STEERING_PART_RE2.stl; visual mesh filename=package://agv_sim/meshes/STEERING_PART_RE2.stl
- link base_link: geometry collision mesh filename=package://agv_sim/meshes/BODY.stl; visual mesh filename=package://agv_sim/meshes/BODY.stl
- link front_wheel_l: geometry collision mesh filename=package://agv_sim/meshes/FRONT_WHEEL_RE2.stl; visual mesh filename=package://agv_sim/meshes/FRONT_WHEEL_RE2.stl
- link front_wheel_r: geometry collision mesh filename=package://agv_sim/meshes/FRONT_WHEEL_RE2.stl; visual mesh filename=package://agv_sim/meshes/FRONT_WHEEL_RE2.stl
- link mast: geometry collision mesh filename=package://agv_sim/meshes/MAST_RE.stl; visual mesh filename=package://agv_sim/meshes/MAST_RE.stl
Joints:
- added joint drive_wheel_joint: type continuous, parent steering_part, child drive_wheel, origin xyz=-0.063 0.012 -0.285 rpy=0 0 0, axis 1 0 0
- added joint steering_joint: type continuous, parent base_link, child steering_part, origin xyz=0.0456 -0.212 0.375 rpy=0 0 0, axis 0 0 1
- joint base_joint: origin xyz=0 0 0.1 rpy=0 0 0 -> xyz=0 0 0 rpy=0 0 0
- joint front_wheel_l_joint: axis 0 1 0 -> 1 0 0
- joint front_wheel_r_joint: axis 0 1 0 -> 1 0 0

File: agv_sim/urdf/agv.urdf copy.xacro (robot description, xacro)
@@ -1,19 +1,4 @@
-<robot name="agv1">
-    <!-- define the material color -->
-    <material name="dark_grey">
-      <color rgba="0.5 0.5 0.5 1.0"/>
-    </material>
-    <material name="orange">
-      <color rgba="0.94 0.38 0.247 1.0"/>
-    </material>
-    <material name="blue">
-      <color rgba="0 0 1.0 1.0"/>
-    </material>
-    <material name="green">
-      <color rgba="0 1.0 0 1.0"/>
-    </material>
-    <material name="white">
-      <color rgba="1.0 1.0 1.0 1.0"/>
-    </material>
+<?xml version="1.0"?>
+<robot xmlns:xacro="http://www.ros.org/wiki/xacro" name="agv1">
   <link name="base_footprint" />
   <joint name="base_joint" type="fixed">
@@ -30,5 +15,5 @@
       <origin xyz="0 0 0" rpy="0 0 0" />
       <geometry>
-        <mesh filename="package://agv_description/meshes/BODY.stl" />
+        <mesh filename="package://agv_sim/meshes/BODY.stl" />
       </geometry>
       <material name="orange" />
@@ -37,5 +22,5 @@
       <origin xyz="0 0 0" rpy="0 0 0" />
       <geometry>
-        <mesh filename="package://agv_description/meshes/BODY.stl" />
+        <mesh filename="package://agv_sim/meshes/BODY.stl" />
       </geometry>
     </collision>
@@ -54,5 +39,5 @@
       <origin xyz="0 0 0" rpy="0 0 0" />
       <geometry>
-        <mesh filename="package://agv_description/meshes/MAST_RE.stl" />
+        <mesh filename="package://agv_sim/meshes/MAST_RE.stl" />
       </geometry>
       <material name="dark_grey" />
@@ -61,5 +46,5 @@
       <origin xyz="0 0 0" rpy="0 0 0" />
       <geometry>
-        <mesh filename="package://agv_description/meshes/MAST_RE.stl" />
+        <mesh filename="package://agv_sim/meshes/MAST_RE.stl" />
       </geometry>
     </collision>
@@ -69,5 +54,5 @@
     <child link="front_wheel_l" />
     <origin xyz="-0.451 0.86 0.035" rpy="0 0 -1.571" />
-    <axis xyz="1 0 0"/>
+    <axis xyz="0 1 0"/>
   </joint>
   <link name="front_wheel_l">
@@ -79,5 +64,5 @@
       <origin xyz="0 0 0" rpy="0 0 0" />
       <geometry>
-        <mesh filename="package://agv_description/meshes/FRONT_WHEEL_RE2.stl"/>
+        <mesh filename="package://agv_sim/meshes/FRONT_WHEEL_RE2.stl"/>
       </geometry>
       <material name="green" />
@@ -86,5 +71,5 @@
       <origin xyz="0 0 0" rpy="0 0 0" />
       <geometry>
-        <mesh filename="package://agv_description/meshes/FRONT_WHEEL_RE2.stl"/>
+        <mesh filename="package://agv_sim/meshes/FRONT_WHEEL_RE2.stl"/>
       </geometry>
     </collision>
@@ -94,5 +79,5 @@
     <child link="front_wheel_r" />
     <origin xyz="0.451 0.86 0.035" rpy="0 0 1.571" />
-    <axis xyz="1 0 0"/>
+    <axis xyz="0 1 0"/>
   </joint>
   <link name="front_wheel_r">
@@ -104,5 +89,5 @@
       <origin xyz="0 0 0" rpy="0 0 0" />
       <geometry>
-        <mesh filename="package://agv_description/meshes/FRONT_WHEEL_RE2.stl"/>
+        <mesh filename="package://agv_sim/meshes/FRONT_WHEEL_RE2.stl"/>
       </geometry>
       <material name="green" />
@@ -111,5 +96,5 @@
       <origin xyz="0 0 0" rpy="0 0 0" />
       <geometry>
-        <mesh filename="package://agv_description/meshes/FRONT_WHEEL_RE2.stl"/>
+        <mesh filename="package://agv_sim/meshes/FRONT_WHEEL_RE2.stl"/>
       </geometry>
     </collision>
@@ -129,12 +114,12 @@
       <origin xyz="0 0 0" rpy="0 0 0" />
       <geometry>
-        <mesh filename="package://agv_description/meshes/STEERING_PART_RE2.stl"/>
+        <mesh filename="package://agv_sim/meshes/STEERING_PART_RE2.stl"/>
       </geometry>
       <material name="white" />
     </visual>
     <collision>
-      <origin xyz="0 0 0" rpy="0 0 0" />
+      <origin xyz="0 0 0" rpy="0 0 3.14" />
       <geometry>
-        <mesh filename="package://agv_description/meshes/STEERING_PART_RE2.stl"/>
+        <mesh filename="package://agv_sim/meshes/STEERING_PART_RE2.stl"/>
       </geometry>
     </collision>
@@ -154,5 +139,5 @@
       <origin xyz="0 0 0" rpy="0 0 0" />
       <geometry>
-        <mesh filename="package://agv_description/meshes/DRIVE_WHEEL_RE2.stl"/>
+        <mesh filename="package://agv_sim/meshes/DRIVE_WHEEL_RE2.stl"/>
       </geometry>
       <material name="blue" />
@@ -161,5 +146,5 @@
       <origin xyz="0 0 0" rpy="0 0 0" />
       <geometry>
-        <mesh filename="package://agv_description/meshes/DRIVE_WHEEL_RE2.stl"/>
+        <mesh filename="package://agv_sim/meshes/DRIVE_WHEEL_RE2.stl"/>
       </geometry>
     </collision>

File: agv_sim/urdf/agv.urdf.xacro (robot description, xacro)
@@ -5,5 +5,5 @@
     <parent link="base_footprint" />
     <child link="base_link" />
-    <origin xyz="0 0 0" rpy="0 0 0" />
+    <origin xyz="0 0 0.1" rpy="0 0 0" />
   </joint>
   <link name="base_link">
@@ -15,5 +15,5 @@
       <origin xyz="0 0 0" rpy="0 0 0" />
       <geometry>
-        <mesh filename="package://agv_description/meshes/BODY.stl" />
+        <mesh filename="package://agv_sim/meshes/BODY.stl" />
       </geometry>
       <material name="orange" />
@@ -22,5 +22,5 @@
       <origin xyz="0 0 0" rpy="0 0 0" />
       <geometry>
-        <mesh filename="package://agv_description/meshes/BODY.stl" />
+        <mesh filename="package://agv_sim/meshes/BODY.stl" />
       </geometry>
     </collision>
@@ -39,5 +39,5 @@
       <origin xyz="0 0 0" rpy="0 0 0" />
       <geometry>
-        <mesh filename="package://agv_description/meshes/MAST_RE.stl" />
+        <mesh filename="package://agv_sim/meshes/MAST_RE.stl" />
       </geometry>
       <material name="dark_grey" />
@@ -46,5 +46,5 @@
       <origin xyz="0 0 0" rpy="0 0 0" />
       <geometry>
-        <mesh filename="package://agv_description/meshes/MAST_RE.stl" />
+        <mesh filename="package://agv_sim/meshes/MAST_RE.stl" />
       </geometry>
     </collision>
@@ -64,5 +64,5 @@
       <origin xyz="0 0 0" rpy="0 0 0" />
       <geometry>
-        <mesh filename="package://agv_description/meshes/FRONT_WHEEL_RE2.stl"/>
+        <mesh filename="package://agv_sim/meshes/FRONT_WHEEL_RE2.stl"/>
       </geometry>
       <material name="green" />
@@ -71,5 +71,5 @@
       <origin xyz="0 0 0" rpy="0 0 0" />
       <geometry>
-        <mesh filename="package://agv_description/meshes/FRONT_WHEEL_RE2.stl"/>
+        <mesh filename="package://agv_sim/meshes/FRONT_WHEEL_RE2.stl"/>
       </geometry>
     </collision>
@@ -89,5 +89,5 @@
       <origin xyz="0 0 0" rpy="0 0 0" />
       <geometry>
-        <mesh filename="package://agv_description/meshes/FRONT_WHEEL_RE2.stl"/>
+        <mesh filename="package://agv_sim/meshes/FRONT_WHEEL_RE2.stl"/>
       </geometry>
       <material name="green" />
@@ -96,37 +96,13 @@
       <origin xyz="0 0 0" rpy="0 0 0" />
       <geometry>
-        <mesh filename="package://agv_description/meshes/FRONT_WHEEL_RE2.stl"/>
+        <mesh filename="package://agv_sim/meshes/FRONT_WHEEL_RE2.stl"/>
       </geometry>
     </collision>
   </link>
-  <joint name="steering_motor_joint" type="continuous">
+  <!-- <joint name="steering_joint" type="continuous">
     <parent link="base_link" />
-    <child link="steering_mortor" />
-    <origin xyz="0.185 -0.2 0.466" rpy="0 0 0" />
+    <child link="steering_part" />
+    <origin xyz="-0.0456 -0.212 0.375" rpy="0 0 0" />
     <axis xyz="0 0 1"/>
-  </joint>
-  <link name="steering_motor">
-    <inertial>
-      <mass value="10"/>
-      <inertia ixx="0.462" ixy="0.0" ixz="-0.002" iyy="0.462" iyz="0.0" izz="0.033"/>
-    </inertial>
-    <visual>
-      <origin xyz="0 0 0" rpy="0 0 0" />
-      <geometry>
-        <mesh filename="package://agv_description/meshes/STEERING_MOTOR.stl" scale="0.001 0.001 0.001"/>
-      </geometry>
-      <material name="white" />
-    </visual>
-    <collision>
-      <origin xyz="0 0 0" rpy="0 0 3.14" />
-      <geometry>
-        <mesh filename="package://agv_description/meshes/STEERING_MOTOR.stl" scale="0.001 0.001 0.001"/>
-      </geometry>
-    </collision>
-  </link>
-  <joint name="steering_joint" type="fixed">
-    <parent link="steering_motor" />
-    <child link="steering_part" />
-    <origin xyz="0.0456 -0.212 0.375" rpy="0 0 0" />
   </joint>
   <link name="steering_part">
@@ -138,12 +114,12 @@
       <origin xyz="0 0 0" rpy="0 0 0" />
       <geometry>
-        <mesh filename="package://agv_description/meshes/STEERING_PART_RE2.stl"/>
+        <mesh filename="package://agv_sim/meshes/STEERING_PART_RE2.stl"/>
       </geometry>
       <material name="white" />
     </visual>
     <collision>
-      <origin xyz="0 0 0" rpy="0 0 3.14" />
+      <origin xyz="0 0 0" rpy="0 0 0" />
       <geometry>
-        <mesh filename="package://agv_description/meshes/STEERING_PART_RE2.stl"/>
+        <mesh filename="package://agv_sim/meshes/STEERING_PART_RE2.stl"/>
       </geometry>
     </collision>
@@ -152,5 +128,5 @@
     <parent link="steering_part" />
     <child link="drive_wheel" />
-    <origin xyz="-0.063 0.012 -0.285" rpy="0 0 0" />
+    <origin xyz="0.063 0.012 -0.285" rpy="0 0 0" />
     <axis xyz="1 0 0"/>
   </joint>
@@ -163,5 +139,5 @@
       <origin xyz="0 0 0" rpy="0 0 0" />
       <geometry>
-        <mesh filename="package://agv_description/meshes/DRIVE_WHEEL_RE2.stl"/>
+        <mesh filename="package://agv_sim/meshes/DRIVE_WHEEL_RE2.stl"/>
       </geometry>
       <material name="blue" />
@@ -170,7 +146,7 @@
       <origin xyz="0 0 0" rpy="0 0 0" />
       <geometry>
-        <mesh filename="package://agv_description/meshes/DRIVE_WHEEL_RE2.stl"/>
+        <mesh filename="package://agv_sim/meshes/DRIVE_WHEEL_RE2.stl"/>
       </geometry>
     </collision>
-  </link>
+  </link> -->
 </robot>

File: agv_sim/urdf/agv1.urdf .xacro (robot description, xacro)
@@ -15,5 +15,5 @@
       <origin xyz="0 0 0" rpy="0 0 0" />
       <geometry>
-        <mesh filename="package://agv_description/meshes/BODY.stl" />
+        <mesh filename="package://agv_sim/meshes/BODY.stl" />
       </geometry>
       <material name="orange" />
@@ -22,5 +22,5 @@
       <origin xyz="0 0 0" rpy="0 0 0" />
       <geometry>
-        <mesh filename="package://agv_description/meshes/BODY.stl" />
+        <mesh filename="package://agv_sim/meshes/BODY.stl" />
       </geometry>
     </collision>
@@ -39,5 +39,5 @@
       <origin xyz="0 0 0" rpy="0 0 0" />
       <geometry>
-        <mesh filename="package://agv_description/meshes/MAST_RE.stl" />
+        <mesh filename="package://agv_sim/meshes/MAST_RE.stl" />
       </geometry>
       <material name="dark_grey" />
@@ -46,5 +46,5 @@
       <origin xyz="0 0 0" rpy="0 0 0" />
       <geometry>
-        <mesh filename="package://agv_description/meshes/MAST_RE.stl" />
+        <mesh filename="package://agv_sim/meshes/MAST_RE.stl" />
       </geometry>
     </collision>
@@ -64,5 +64,5 @@
       <origin xyz="0 0 0" rpy="0 0 0" />
       <geometry>
-        <mesh filename="package://agv_description/meshes/FRONT_WHEEL_RE2.stl"/>
+        <mesh filename="package://agv_sim/meshes/FRONT_WHEEL_RE2.stl"/>
       </geometry>
       <material name="green" />
@@ -71,5 +71,5 @@
       <origin xyz="0 0 0" rpy="0 0 0" />
       <geometry>
-        <mesh filename="package://agv_description/meshes/FRONT_WHEEL_RE2.stl"/>
+        <mesh filename="package://agv_sim/meshes/FRONT_WHEEL_RE2.stl"/>
       </geometry>
     </collision>
@@ -89,5 +89,5 @@
       <origin xyz="0 0 0" rpy="0 0 0" />
       <geometry>
-        <mesh filename="package://agv_description/meshes/FRONT_WHEEL_RE2.stl"/>
+        <mesh filename="package://agv_sim/meshes/FRONT_WHEEL_RE2.stl"/>
       </geometry>
       <material name="green" />
@@ -96,23 +96,23 @@
       <origin xyz="0 0 0" rpy="0 0 0" />
       <geometry>
-        <mesh filename="package://agv_description/meshes/FRONT_WHEEL_RE2.stl"/>
+        <mesh filename="package://agv_sim/meshes/FRONT_WHEEL_RE2.stl"/>
       </geometry>
     </collision>
   </link>
-  <joint name="steering_joint" type="continuous">
+  <joint name="steering_motor_joint" type="continuous">
     <parent link="base_link" />
-    <child link="steering_part" />
-    <origin xyz="0.0456 -0.212 0.375" rpy="0 0 0" />
+    <child link="steering_mortor" />
+    <origin xyz="0.185 -0.2 0.466" rpy="0 0 0" />
     <axis xyz="0 0 1"/>
   </joint>
-  <link name="steering_part">
+  <link name="steering_motor">
     <inertial>
-      <mass value="85.197"/>
-      <inertia ixx="2.8" ixy="0.0" ixz="0.11" iyy="2.84" iyz="-0.11" izz="0.93"/>
+      <mass value="10"/>
+      <inertia ixx="0.462" ixy="0.0" ixz="-0.002" iyy="0.462" iyz="0.0" izz="0.033"/>
     </inertial>
     <visual>
       <origin xyz="0 0 0" rpy="0 0 0" />
       <geometry>
-        <mesh filename="package://agv_description/meshes/STEERING_PART_RE2.stl"/>
+        <mesh filename="package://agv_sim/meshes/STEERING_MOTOR.stl" scale="0.001 0.001 0.001"/>
       </geometry>
       <material name="white" />
@@ -121,5 +121,29 @@
       <origin xyz="0 0 0" rpy="0 0 3.14" />
       <geometry>
-        <mesh filename="package://agv_description/meshes/STEERING_PART_RE2.stl"/>
+        <mesh filename="package://agv_sim/meshes/STEERING_MOTOR.stl" scale="0.001 0.001 0.001"/>
+      </geometry>
+    </collision>
+  </link>
+  <joint name="steering_joint" type="fixed">
+    <parent link="steering_motor" />
+    <child link="steering_part" />
+    <origin xyz="0.0456 -0.212 0.375" rpy="0 0 0" />
+  </joint>
+  <link name="steering_part">
+    <inertial>
+      <mass value="85.056"/>
+      <inertia ixx="2.77" ixy="0.0" ixz="0.12" iyy="2.81" iyz="-0.11" izz="0.9"/>
+    </inertial>
+    <visual>
+      <origin xyz="0 0 0" rpy="0 0 0" />
+      <geometry>
+        <mesh filename="package://agv_sim/meshes/STEERING_PART_RE2.stl"/>
+      </geometry>
+      <material name="white" />
+    </visual>
+    <collision>
+      <origin xyz="0 0 0" rpy="0 0 3.14" />
+      <geometry>
+        <mesh filename="package://agv_sim/meshes/STEERING_PART_RE2.stl"/>
       </geometry>
     </collision>
@@ -134,10 +158,10 @@
     <inertial>
       <mass value="21.755"/>
-      <inertia ixx="2.03" ixy="0.02" ixz="-0.42" iyy="2.03" iyz="-0.07" izz="0.27"/>
+      <inertia ixx="0.265" ixy="0.0" ixz="0.0" iyy="0.166" iyz="0.0" izz="0.166"/>
     </inertial>
     <visual>
       <origin xyz="0 0 0" rpy="0 0 0" />
       <geometry>
-        <mesh filename="package://agv_description/meshes/DRIVE_WHEEL_RE2.stl"/>
+        <mesh filename="package://agv_sim/meshes/DRIVE_WHEEL_RE2.stl"/>
       </geometry>
       <material name="blue" />
@@ -146,5 +170,5 @@
       <origin xyz="0 0 0" rpy="0 0 0" />
       <geometry>
-        <mesh filename="package://agv_description/meshes/DRIVE_WHEEL_RE2.stl"/>
+        <mesh filename="package://agv_sim/meshes/DRIVE_WHEEL_RE2.stl"/>
       </geometry>
     </collision>

File: agv_sim/urdf/demo.urdf.xacro (robot description, xacro)
@@ -18,5 +18,5 @@
   </material>
   <!-- this include provides the macro definition used below -->
- <xacro:include filename="$(find agv_description)/urdf/agv.urdf.xacro"/>
+ <xacro:include filename="$(find agv_sim)/urdf/agv.urdf.xacro"/>
  <xacro:property name="model" value="(arg model)"/>
  <!-- if more models are defined, add them here -->

Commit message: fake node를 이용하여 직접 구상한 컨트롤 매소드로 rviz2상에서 agv 시뮬레이션

File: agv_sim/urdf/agv.urdf (robot description, URDF)
Before this commit: robot agv1, 7 links, 6 joints
Joints:
- joint front_wheel_l_joint: type continuous -> fixed
- joint front_wheel_r_joint: type continuous -> fixed

File: agv_sim/urdf/agv.urdf.xacro (robot description, xacro)
@@ -100,5 +100,5 @@
     </collision>
   </link>
-  <!-- <joint name="steering_joint" type="continuous">
+  <joint name="steering_joint" type="continuous">
     <parent link="base_link" />
     <child link="steering_part" />
@@ -149,29 +149,25 @@
       </geometry>
     </collision>
-  </link> -->
-  <joint name="drive_wheel_joint" type="continuous">
-    <parent link="base_link" />
-    <child link="drive_wheel" />
-    <origin xyz="0.0174 -0.2 0.09" rpy="0 0 0" />
-    <axis xyz="1 0 0"/>
-  </joint>
-  <link name="drive_wheel">
-    <inertial>
-      <mass value="21.755"/>
-      <inertia ixx="0.265" ixy="0.0" ixz="0.0" iyy="0.166" iyz="0.0" izz="0.166"/>
-    </inertial>
-    <visual>
-      <origin xyz="0 0 0" rpy="0 0 0" />
-      <geometry>
-        <mesh filename="package://agv_sim/meshes/DRIVE_WHEEL_RE2.stl"/>
-      </geometry>
-      <material name="blue" />
-    </visual>
-    <collision>
-      <origin xyz="0 0 0" rpy="0 0 0" />
-      <geometry>
-        <mesh filename="package://agv_sim/meshes/DRIVE_WHEEL_RE2.stl"/>
-      </geometry>
-    </collision>
   </link>
+  <!-- <gazebo>
+    <plugin name="agv_drive" filename="libgazebo_ros_tricycle_drive.so">
+      <robotNameSpace>/agv1</robotNameSpace>
+      <update_rate>30</update_rate>
+      <steering_joint>steering_joint</steering_joint>
+      <actuated_wheel_joint>drive_wheel_joint</actuated_wheel_joint>
+      <encoder_wheel_left_joint>front_wheel_l_joint</encoder_wheel_left_joint>
+      <encoder_wheel_right_joint>front_wheel_r_joint</encoder_wheel_right_joint>
+      <wheel_separation>0.9</wheel_separation>
+      <encoder_wheel_diameter>0.25</encoder_wheel_diameter>
+      <actuated_wheel_diameter>0.31</actuated_wheel_diameter>
+      <max_wheel_torque>100</max_wheel_torque>
+      <max_wheel_acceleration>5.0</max_wheel_acceleration>
+      <max_steering_speed>1.0</max_steering_speed>
+      <publish_odom>true</publish_odom>
+      <publish_wheel_tf>true</publish_wheel_tf>
+      <publish_wheel_joint_state>true</publish_wheel_joint_state>
+      <odometry_frame>odom</odometry_frame>
+      <robot_base_frame>base_footprint</robot_base_frame>
+    </plugin>
+  </gazebo> -->
 </robot>
