Commit message: 패키지 정리

File: agv_sim/urdf/agv.urdf.xacro (robot description, xacro)
@@ -39,5 +39,5 @@
       <origin xyz="0 0 0" rpy="0 0 0" />
       <geometry>
-        <mesh filename="package://agv_sim/meshes/MAST_RE.stl" />
+        <mesh filename="package://agv_sim/meshes/MAST.stl" scale = "0.001 0.001 0.001" />
       </geometry>
       <material name="dark_grey" />
@@ -46,5 +46,5 @@
       <origin xyz="0 0 0" rpy="0 0 0" />
       <geometry>
-        <mesh filename="package://agv_sim/meshes/MAST_RE.stl" />
+        <mesh filename="package://agv_sim/meshes/MAST.stl" scale = "0.001 0.001 0.001" />
       </geometry>
     </collision>
@@ -100,5 +100,5 @@
     </collision>
   </link>
-  <!-- <joint name="steering_joint" type="continuous">
+  <joint name="steering_joint" type="continuous">
     <parent link="base_link" />
     <child link="steering_part" />
@@ -149,4 +149,4 @@
       </geometry>
     </collision>
-  </link> -->
+  </link>
 </robot>

File: agv_sim/urdf/agv1.urdf .xacro (robot description, xacro)
@@ -5,5 +5,5 @@
     <parent link="base_footprint" />
     <child link="base_link" />
-    <origin xyz="0 0 0" rpy="0 0 0" />
+    <origin xyz="0 0 0.11" rpy="0 0 0" />
   </joint>
   <link name="base_link">
@@ -39,5 +39,5 @@
       <origin xyz="0 0 0" rpy="0 0 0" />
       <geometry>
-        <mesh filename="package://agv_sim/meshes/MAST_RE.stl" />
+        <mesh filename="package://agv_sim/meshes/MAST.stl" scale = "0.001 0.001 0.001" />
       </geometry>
       <material name="dark_grey" />
@@ -46,5 +46,5 @@
       <origin xyz="0 0 0" rpy="0 0 0" />
       <geometry>
-        <mesh filename="package://agv_sim/meshes/MAST_RE.stl" />
+        <mesh filename="package://agv_sim/meshes/MAST.stl" scale = "0.001 0.001 0.001" />
       </geometry>
     </collision>
@@ -100,31 +100,6 @@
     </collision>
   </link>
-  <joint name="steering_motor_joint" type="continuous">
+  <joint name="steering_joint" type="continuos">
     <parent link="base_link" />
-    <child link="steering_mortor" />
-    <origin xyz="0.185 -0.2 0.466" rpy="0 0 0" />
-    <axis xyz="0 0 1"/>
-  </joint>
-  <link name="steering_motor">
-    <inertial>
-      <mass value="10"/>
-      <inertia ixx="0.462" ixy="0.0" ixz="-0.002" iyy="0.462" iyz="0.0" izz="0.033"/>
-    </inertial>
-    <visual>
-      <origin xyz="0 0 0" rpy="0 0 0" />
-      <geometry>
-        <mesh filename="package://agv_sim/meshes/STEERING_MOTOR.stl" scale="0.001 0.001 0.001"/>
-      </geometry>
-      <material name="white" />
-    </visual>
-    <collision>
-      <origin xyz="0 0 0" rpy="0 0 3.14" />
-      <geometry>
-        <mesh filename="package://agv_sim/meshes/STEERING_MOTOR.stl" scale="0.001 0.001 0.001"/>
-      </geometry>
-    </collision>
-  </link>
-  <joint name="steering_joint" type="fixed">
-    <parent link="steering_motor" />
     <child link="steering_part" />
     <origin xyz="0.0456 -0.212 0.375" rpy="0 0 0" />

Commit message: gazebo plugin 미적용 및 적용 합본 백업

File: agv_sim/urdf/agv.urdf.xacro (robot description, xacro)
@@ -100,5 +100,5 @@
     </collision>
   </link>
-  <joint name="steering_joint" type="continuous">
+  <!-- <joint name="steering_joint" type="continuous">
     <parent link="base_link" />
     <child link="steering_part" />
@@ -149,4 +149,29 @@
       </geometry>
     </collision>
+  </link> -->
+  <joint name="drive_wheel_joint" type="continuous">
+    <parent link="base_link" />
+    <child link="drive_wheel" />
+    <origin xyz="0.0174 -0.2 0.09" rpy="0 0 0" />
+    <axis xyz="1 0 0"/>
+  </joint>
+  <link name="drive_wheel">
+    <inertial>
+      <mass value="21.755"/>
+      <inertia ixx="0.265" ixy="0.0" ixz="0.0" iyy="0.166" iyz="0.0" izz="0.166"/>
+    </inertial>
+    <visual>
+      <origin xyz="0 0 0" rpy="0 0 0" />
+      <geometry>
+        <mesh filename="package://agv_sim/meshes/DRIVE_WHEEL_RE2.stl"/>
+      </geometry>
+      <material name="blue" />
+    </visual>
+    <collision>
+      <origin xyz="0 0 0" rpy="0 0 0" />
+      <geometry>
+        <mesh filename="package://agv_sim/meshes/DRIVE_WHEEL_RE2.stl"/>
+      </geometry>
+    </collision>
   </link>
 </robot>

File: agv_sim/urdf/agv_plug.urdf.xacro (robot description, xacro)
@@ -5,5 +5,5 @@
     <parent link="base_footprint" />
     <child link="base_link" />
-    <origin xyz="0 0 0.11" rpy="0 0 0" />
+    <origin xyz="0 0 0.1" rpy="0 0 0" />
   </joint>
   <link name="base_link">
@@ -100,8 +100,8 @@
     </collision>
   </link>
-  <joint name="steering_joint" type="continuos">
+  <joint name="steering_joint" type="continuous">
     <parent link="base_link" />
     <child link="steering_part" />
-    <origin xyz="0.0456 -0.212 0.375" rpy="0 0 0" />
+    <origin xyz="-0.0456 -0.212 0.375" rpy="0 0 0" />
     <axis xyz="0 0 1"/>
   </joint>
@@ -119,5 +119,5 @@
     </visual>
     <collision>
-      <origin xyz="0 0 0" rpy="0 0 3.14" />
+      <origin xyz="0 0 0" rpy="0 0 0" />
       <geometry>
         <mesh filename="package://agv_sim/meshes/STEERING_PART_RE2.stl"/>
@@ -128,5 +128,5 @@
     <parent link="steering_part" />
     <child link="drive_wheel" />
-    <origin xyz="-0.063 0.012 -0.285" rpy="0 0 0" />
+    <origin xyz="0.063 0.012 -0.285" rpy="0 0 0" />
     <axis xyz="1 0 0"/>
   </joint>

Commit message: gazebo_plugin 제작 시작

File: agv_sim/urdf/agv.urdf.xacro (robot description, xacro)
@@ -50,5 +50,5 @@
     </collision>
   </link>
-  <joint name="front_wheel_l_joint" type="continuous">
+  <joint name="front_wheel_l_joint" type="fixed">
     <parent link="base_link" />
     <child link="front_wheel_l" />
@@ -75,5 +75,5 @@
     </collision>
   </link>
-  <joint name="front_wheel_r_joint" type="continuous">
+  <joint name="front_wheel_r_joint" type="fixed">
     <parent link="base_link" />
     <child link="front_wheel_r" />
@@ -150,5 +150,26 @@
     </collision>
   </link>
-  <!-- <gazebo>
+  <gazebo>
+    <plugin name="gazebo_ros2_control" filename="libgazebo_ros2_control.so"/>
+  </gazebo>
+  <ros2_control name="MyRobotController" type="system">
+    <hardware>
+      <plugin>gazebo_ros2_control/GazeboSystem</plugin>
+      <!-- Optionally, specify additional plugin parameters -->
+    </hardware>
+    <joint>
+      <name>steering_joint</name>
+      <command_interface>position</command_interface>
+      <state_interface>position</state_interface>
+      <state_interface>velocity</state_interface>
+    </joint>
+    <joint>
+      <name>drive_wheel_joint</name>
+      <command_interface>position</command_interface>
+      <state_interface>position</state_interface>
+      <state_interface>velocity</state_interface>
+    </joint>
+  </ros2_control>
+  <gazebo>
     <plugin name="agv_drive" filename="libgazebo_ros_tricycle_drive.so">
       <robotNameSpace>/agv1</robotNameSpace>
@@ -170,4 +191,4 @@
       <robot_base_frame>base_footprint</robot_base_frame>
     </plugin>
-  </gazebo> -->
+  </gazebo>
 </robot>

File: agv_sim/urdf/agv1.urdf .xacro (robot description, xacro)
@@ -50,5 +50,5 @@
     </collision>
   </link>
-  <joint name="front_wheel_l_joint" type="continuous">
+  <joint name="front_wheel_l_joint" type="fixed">
     <parent link="base_link" />
     <child link="front_wheel_l" />
@@ -75,5 +75,5 @@
     </collision>
   </link>
-  <joint name="front_wheel_r_joint" type="continuous">
+  <joint name="front_wheel_r_joint" type="fixed">
     <parent link="base_link" />
     <child link="front_wheel_r" />

Commit message: gazebo_agv_drive_plugin 제작 - 캐스터 조인트 제거중

File: agv_sim/urdf/agv.urdf.xacro (robot description, xacro)
@@ -15,5 +15,5 @@
       <origin xyz="0 0 0" rpy="0 0 0" />
       <geometry>
-        <mesh filename="package://agv_sim/meshes/BODY.stl" />
+        <mesh filename="package://agv_sim/meshes/BODY_RE5.stl" scale = "0.001 0.001 0.001"/>
       </geometry>
       <material name="orange" />
@@ -22,9 +22,9 @@
       <origin xyz="0 0 0" rpy="0 0 0" />
       <geometry>
-        <mesh filename="package://agv_sim/meshes/BODY.stl" />
+        <mesh filename="package://agv_sim/meshes/BODY_RE5.stl" scale = "0.001 0.001 0.001" />
       </geometry>
     </collision>
   </link>
-  <joint name="mast_joint" type="fixed">
+  <!-- <joint name="mast_joint" type="fixed">
     <parent link="base_link" />
     <child link="mast" />
@@ -99,6 +99,6 @@
       </geometry>
     </collision>
-  </link>
-  <joint name="steering_joint" type="continuous">
+  </link> -->
+  <joint name="steering_joint" type="fixed">
     <parent link="base_link" />
     <child link="steering_part" />
@@ -150,5 +150,5 @@
     </collision>
   </link>
-  <gazebo>
+  <!-- <gazebo>
     <plugin name="gazebo_ros2_control" filename="libgazebo_ros2_control.so"/>
   </gazebo>
@@ -156,5 +156,4 @@
     <hardware>
       <plugin>gazebo_ros2_control/GazeboSystem</plugin>
-      <!-- Optionally, specify additional plugin parameters -->
     </hardware>
     <joint>
@@ -170,6 +169,6 @@
       <state_interface>velocity</state_interface>
     </joint>
-  </ros2_control>
-  <gazebo>
+  </ros2_control> -->
+  <!-- <gazebo>
     <plugin name="agv_drive" filename="libgazebo_ros_tricycle_drive.so">
       <robotNameSpace>/agv1</robotNameSpace>
@@ -191,4 +190,4 @@
       <robot_base_frame>base_footprint</robot_base_frame>
     </plugin>
-  </gazebo>
+  </gazebo> -->
 </robot>

Commit message: gazebo_plugin - drive_wheel 기반 - steering_joint 미반영

File: agv_sim/urdf/agv.urdf.xacro (robot description, xacro)
@@ -15,5 +15,5 @@
       <origin xyz="0 0 0" rpy="0 0 0" />
       <geometry>
-        <mesh filename="package://agv_sim/meshes/BODY_RE5.stl" scale = "0.001 0.001 0.001"/>
+        <mesh filename="package://agv_sim/meshes/BODY.stl" />
       </geometry>
       <material name="orange" />
@@ -22,5 +22,5 @@
       <origin xyz="0 0 0" rpy="0 0 0" />
       <geometry>
-        <mesh filename="package://agv_sim/meshes/BODY_RE5.stl" scale = "0.001 0.001 0.001" />
+        <mesh filename="package://agv_sim/meshes/BODY.stl"  />
       </geometry>
     </collision>
@@ -49,6 +49,6 @@
       </geometry>
     </collision>
-  </link>
-  <joint name="front_wheel_l_joint" type="fixed">
+  </link> -->
+  <joint name="front_wheel_l_joint" type="continuous">
     <parent link="base_link" />
     <child link="front_wheel_l" />
@@ -75,5 +75,5 @@
     </collision>
   </link>
-  <joint name="front_wheel_r_joint" type="fixed">
+  <joint name="front_wheel_r_joint" type="continuous">
     <parent link="base_link" />
     <child link="front_wheel_r" />
@@ -99,5 +99,5 @@
       </geometry>
     </collision>
-  </link> -->
+  </link>
   <joint name="steering_joint" type="fixed">
     <parent link="base_link" />

File: agv_sim/urdf/agv1.urdf .xacro (robot description, xacro)
@@ -17,5 +17,5 @@
         <mesh filename="package://agv_sim/meshes/BODY.stl" />
       </geometry>
-      <material name="orange" />
+      <material name="orange"/>
     </visual>
     <collision>

Commit message: 시뮬레이션에서 LiDAR 및 환경 기본 구축

File: agv_sim/urdf/agv.urdf.xacro (robot description, xacro)
@@ -150,44 +150,77 @@
     </collision>
   </link>
-  <!-- <gazebo>
-    <plugin name="gazebo_ros2_control" filename="libgazebo_ros2_control.so"/>
-  </gazebo>
-  <ros2_control name="MyRobotController" type="system">
-    <hardware>
-      <plugin>gazebo_ros2_control/GazeboSystem</plugin>
-    </hardware>
-    <joint>
-      <name>steering_joint</name>
-      <command_interface>position</command_interface>
-      <state_interface>position</state_interface>
-      <state_interface>velocity</state_interface>
-    </joint>
-    <joint>
-      <name>drive_wheel_joint</name>
-      <command_interface>position</command_interface>
-      <state_interface>position</state_interface>
-      <state_interface>velocity</state_interface>
-    </joint>
-  </ros2_control> -->
-  <!-- <gazebo>
-    <plugin name="agv_drive" filename="libgazebo_ros_tricycle_drive.so">
-      <robotNameSpace>/agv1</robotNameSpace>
-      <update_rate>30</update_rate>
-      <steering_joint>steering_joint</steering_joint>
-      <actuated_wheel_joint>drive_wheel_joint</actuated_wheel_joint>
-      <encoder_wheel_left_joint>front_wheel_l_joint</encoder_wheel_left_joint>
-      <encoder_wheel_right_joint>front_wheel_r_joint</encoder_wheel_right_joint>
-      <wheel_separation>0.9</wheel_separation>
-      <encoder_wheel_diameter>0.25</encoder_wheel_diameter>
-      <actuated_wheel_diameter>0.31</actuated_wheel_diameter>
-      <max_wheel_torque>100</max_wheel_torque>
-      <max_wheel_acceleration>5.0</max_wheel_acceleration>
-      <max_steering_speed>1.0</max_steering_speed>
-      <publish_odom>true</publish_odom>
-      <publish_wheel_tf>true</publish_wheel_tf>
-      <publish_wheel_joint_state>true</publish_wheel_joint_state>
-      <odometry_frame>odom</odometry_frame>
-      <robot_base_frame>base_footprint</robot_base_frame>
-    </plugin>
-  </gazebo> -->
+  <joint name="slam_lidar_joint" type="fixed">
+    <parent link="base_link" />
+    <child link="slam_lidar" />
+    <origin xyz="0 -0.2 2.149" rpy="0 0 0" />
+  </joint>
+  <link name="slam_lidar">
+    <inertial>
+      <mass value="0.641"/>
+      <inertia ixx="0.0" ixy="0.0" ixz="0.0" iyy="0.0" iyz="0.0" izz="0.0"/>
+    </inertial>
+    <visual>
+      <origin xyz="0 0 0" rpy="0 0 0" />
+      <geometry>
+        <mesh filename="package://agv_sim/meshes/3D_SLAM_LIDAR.stl" scale = "0.001 0.001 0.001"/>
+      </geometry>
+    </visual>
+    <!-- <collision>
+      <origin xyz="0 0 0" rpy="0 0 0" />
+      <geometry>
+        <mesh filename="package://agv_sim/meshes/3D_SLAM_LIDAR.stl" scale = "0.001 0.001 0.001"/>
+      </geometry>
+    </collision> -->
+  </link>
+  <joint name="safety_lidar_l_joint" type="fixed">
+    <parent link="base_link" />
+    <child link="safety_lidar_l" />
+    <origin xyz="-0.442 -0.332 0.004" rpy="0 0 -2.3562" />
+  </joint>
+  <link name="safety_lidar_l">
+    <inertial>
+      <mass value="0"/>
+      <inertia ixx="0.0" ixy="0.0" ixz="0.0" iyy="0.0" iyz="0.0" izz="0.0"/>
+    </inertial>
+    <visual>
+      <origin xyz="0 0 0" rpy="-1.57 0 1.57" />
+      <geometry>
+        <mesh filename="package://agv_sim/meshes/2D_SAFETY_LIDAR.stl" scale = "0.001 0.001 0.001"/>
+      </geometry>
+    </visual>
+  </link>
+  <joint name="safety_lidar_r_joint" type="fixed">
+    <parent link="base_link" />
+    <child link="safety_lidar_r" />
+    <origin xyz="0.442 -0.332 0.004" rpy="0 0 -0.7854" />
+  </joint>
+  <link name="safety_lidar_r">
+    <inertial>
+      <mass value="0"/>
+      <inertia ixx="0.0" ixy="0.0" ixz="0.0" iyy="0.0" iyz="0.0" izz="0.0"/>
+    </inertial>
+    <visual>
+      <origin xyz="0 0 0" rpy="-1.57 0 1.56" />
+      <geometry>
+        <mesh filename="package://agv_sim/meshes/2D_SAFETY_LIDAR.stl" scale = "0.001 0.001 0.001"/>
+      </geometry>
+    </visual>
+  </link>
+  <joint name="safety_lidar_m_joint" type="fixed">
+    <parent link="base_link" />
+    <child link="safety_lidar_m" />
+    <origin xyz="0 0.863 0" rpy="0 0 1.57" />
+  </joint>
+  <link name="safety_lidar_m">
+    <inertial>
+      <mass value="0"/>
+      <inertia ixx="0.0" ixy="0.0" ixz="0.0" iyy="0.0" iyz="0.0" izz="0.0"/>
+    </inertial>
+    <visual>
+      <origin xyz="0 0 0" rpy="-1.57 0 1.57" />
+      <geometry>
+        <mesh filename="package://agv_sim/meshes/2D_SAFETY_LIDAR.stl" scale = "0.001 0.001 0.001"/>
+      </geometry>
+    </visual>
+  </link>
 </robot>

Commit message: Gazebo LiDAR 입력 완료

File: agv_sim/urdf/agv.urdf.xacro (robot description, xacro)
@@ -153,5 +153,5 @@
     <parent link="base_link" />
     <child link="slam_lidar" />
-    <origin xyz="0 -0.2 2.149" rpy="0 0 0" />
+    <origin xyz="0 -0.2 2.207" rpy="0 0 0" />
   </joint>
   <link name="slam_lidar">
@@ -163,5 +163,5 @@
       <origin xyz="0 0 0" rpy="0 0 0" />
       <geometry>
-        <mesh filename="package://agv_sim/meshes/3D_SLAM_LIDAR.stl" scale = "0.001 0.001 0.001"/>
+        <mesh filename="package://agv_sim/meshes/C16_3D.stl" scale = "0.001 0.001 0.001"/>
       </geometry>
     </visual>
