Commit message: - 로봇 축 변경  전방 y축 -> x축

File: agv_sim/urdf/modified_agv.urdf.xacro (robot description, xacro)
@@ -9,9 +9,10 @@
   <link name="base_link">
     <inertial>
+      <origin xyz="0 0 0.89" rpy="0 0 0"/>
       <mass value="2129.355" />
-      <inertia ixx="962.268" ixy="-2.68" ixz="13.459" iyy="963.850" iyz="81.387" izz="482.35" />
-    </inertial>
-    <visual>
-      <origin xyz="0 0 0" rpy="0 0 0" />
+      <inertia ixx="990" ixy="0" ixz="0" iyy="990" iyz="0" izz="990" />
+    </inertial>
+    <visual>
+      <origin xyz="0 0 0" rpy="0 0 1.574" />
       <geometry>
         <mesh filename="package://agv_sim/meshes/BODY.stl" />
@@ -20,5 +21,5 @@
     </visual>
     <collision>
-      <origin xyz="0 0 0" rpy="0 0 0" />
+      <origin xyz="0 0 0" rpy="0 0 1.574" />
       <geometry>
         <mesh filename="package://agv_sim/meshes/BODY.stl"  />
@@ -53,5 +54,5 @@
     <parent link="base_link" />
     <child link="steering_part" />
-    <origin xyz="-0.0456 -0.212 0.375" rpy="0 0 0" />
+    <origin xyz="0.212 -0.0456 0.375" rpy="0 0 1.574" />
     <axis xyz="0 0 1"/>
   </joint>
@@ -59,5 +60,5 @@
     <inertial>
       <mass value="85.056"/>
-      <inertia ixx="2.77" ixy="0.0" ixz="0.12" iyy="2.81" iyz="-0.11" izz="0.9"/>
+      <inertia ixx="2.81" ixy="0.0" ixz="-0.11" iyy="2.77" iyz="0.12" izz="0.9"/>
     </inertial>
     <visual>
@@ -84,5 +85,5 @@
     <inertial>
       <mass value="21.755"/>
-      <inertia ixx="0.265" ixy="0.0" ixz="0.0" iyy="0.166" iyz="0.0" izz="0.166"/>
+      <inertia ixx="0.166" ixy="0.0" ixz="0.0" iyy="0.166" iyz="0.0" izz="0.166"/>
     </inertial>
     <visual>
@@ -103,5 +104,5 @@
     <parent link="base_link" />
     <child link="front_wheel_l" />
-    <origin xyz="-0.451 0.86 0.035" rpy="0 0 -1.571" />
+    <origin xyz="-0.86 -0.451 0.035" rpy="0 0 0" />
     <axis xyz="0 1 0"/>
   </joint>
@@ -109,5 +110,5 @@
     <inertial>
       <mass value="16.096"/>
-      <inertia ixx="0.066" ixy="0.0" ixz="0.0" iyy="0.104" iyz="0.0" izz="0.066"/>
+      <inertia ixx="0.066" ixy="0.0" ixz="0.0" iyy="0.066" iyz="0.0" izz="0.066"/>
     </inertial>
     <visual>
@@ -128,5 +129,5 @@
     <parent link="base_link" />
     <child link="front_wheel_r" />
-    <origin xyz="0.451 0.86 0.035" rpy="0 0 1.571" />
+    <origin xyz="-0.86 0.451 0.035" rpy="0 0 3.14" />
     <axis xyz="0 1 0"/>
   </joint>
@@ -134,5 +135,5 @@
     <inertial>
       <mass value="16.096"/>
-      <inertia ixx="0.066" ixy="0.0" ixz="0.0" iyy="0.104" iyz="0.0" izz="0.066"/>
+      <inertia ixx="0.066" ixy="0.0" ixz="0.0" iyy="0.066" iyz="0.0" izz="0.066"/>
     </inertial>
     <visual>
@@ -153,5 +154,5 @@
     <parent link="base_link"/>
     <child link="imu_link"/>
-    <origin xyz="0.103 0.341 0.873" rpy="0 0 -1.574"/>
+    <origin xyz="-0.341 0.103 0.873" rpy="0 0 0"/>
   </joint>
   <link name="imu_link"/>
@@ -176,5 +177,5 @@
     <parent link="base_link" />
     <child link="safety_lidar_l" />
-    <origin xyz="-0.442 -0.332 0.004" rpy="0 0 -2.3562" />
+    <origin xyz="0.332 -0.442 0.004" rpy="0 0 -0.7854" />
   </joint>
   <link name="safety_lidar_l">
@@ -193,5 +194,5 @@
     <parent link="base_link" />
     <child link="safety_lidar_r" />
-    <origin xyz="0.442 -0.332 0.004" rpy="0 0 -0.7854" />
+    <origin xyz="0.332 0.442 0.004" rpy="0 0 0.7854" />
   </joint>
   <link name="safety_lidar_r">
@@ -210,5 +211,5 @@
     <parent link="base_link" />
     <child link="safety_lidar_m" />
-    <origin xyz="0 0.863 0" rpy="0 0 1.57" />
+    <origin xyz="-0.863 0 0" rpy="0 0 3.14" />
   </joint>
   <link name="safety_lidar_m">

Commit message: slam 조정

File: agv_sim/urdf/modified_agv.urdf.xacro (robot description, xacro)
@@ -51,8 +51,8 @@
     </collision>
   </link> -->
-  <joint name="steering_joint" type="fixed">
+  <joint name="steering_joint" type="continuous">
     <parent link="base_link" />
     <child link="steering_part" />
-    <origin xyz="0.212 -0.0456 0.375" rpy="0 0 1.574" />
+    <origin xyz="0.212 -0.0456 0.344" rpy="0 0 1.574" />
     <axis xyz="0 0 1"/>
   </joint>
@@ -104,5 +104,5 @@
     <parent link="base_link" />
     <child link="front_wheel_l" />
-    <origin xyz="-0.86 -0.451 0.035" rpy="0 0 0" />
+    <origin xyz="-0.86 -0.451 0.025" rpy="0 0 0" />
     <axis xyz="0 1 0"/>
   </joint>
@@ -129,5 +129,5 @@
     <parent link="base_link" />
     <child link="front_wheel_r" />
-    <origin xyz="-0.86 0.451 0.035" rpy="0 0 3.14" />
+    <origin xyz="-0.86 0.451 0.025" rpy="0 0 3.14" />
     <axis xyz="0 1 0"/>
   </joint>
@@ -154,5 +154,5 @@
     <parent link="base_link"/>
     <child link="imu_link"/>
-    <origin xyz="-0.341 0.103 0.873" rpy="0 0 0"/>
+    <origin xyz="-0.341 0.103 0.763" rpy="0 0 0"/>
   </joint>
   <link name="imu_link"/>
@@ -160,5 +160,5 @@
     <parent link="base_link" />
     <child link="slam_lidar" />
-    <origin xyz="0 -0.2 2.207" rpy="0 0 0" />
+    <origin xyz="0 -0.2 2.197" rpy="0 0 0" />
   </joint>
   <link name="slam_lidar">
@@ -177,5 +177,5 @@
     <parent link="base_link" />
     <child link="safety_lidar_l" />
-    <origin xyz="0.332 -0.442 0.004" rpy="0 0 -0.7854" />
+    <origin xyz="0.332 -0.442 -0.006" rpy="0 0 -0.7854" />
   </joint>
   <link name="safety_lidar_l">
@@ -194,5 +194,5 @@
     <parent link="base_link" />
     <child link="safety_lidar_r" />
-    <origin xyz="0.332 0.442 0.004" rpy="0 0 0.7854" />
+    <origin xyz="0.332 0.442 -0.006" rpy="0 0 0.7854" />
   </joint>
   <link name="safety_lidar_r">
@@ -211,5 +211,5 @@
     <parent link="base_link" />
     <child link="safety_lidar_m" />
-    <origin xyz="-0.863 0 0" rpy="0 0 3.14" />
+    <origin xyz="-0.863 0 -0.01" rpy="0 0 3.14" />
   </joint>
   <link name="safety_lidar_m">

Commit message: slam 테스트중

File: agv_sim/urdf/modified_agv.urdf.xacro (robot description, xacro)
@@ -54,5 +54,5 @@
     <parent link="base_link" />
     <child link="steering_part" />
-    <origin xyz="0.212 -0.0456 0.344" rpy="0 0 1.574" />
+    <origin xyz="0.212 -0.0476 0.344" rpy="0 0 1.574" />
     <axis xyz="0 0 1"/>
   </joint>

Commit message: 드라이빙 플러그인 수정 - imu 추가 - 스티어링 추가
cartographer 기반 SLAM 적용

File: agv_sim/urdf/modified_agv.urdf.xacro (robot description, xacro)
@@ -54,5 +54,6 @@
     <parent link="base_link" />
     <child link="steering_part" />
-    <origin xyz="0.212 -0.0476 0.344" rpy="0 0 1.574" />
+    <origin xyz="0.216 0 0.344" rpy="0 0 1.574" />
+    <!-- 0.212 -0.0476 0.344 -->
     <axis xyz="0 0 1"/>
   </joint>
@@ -65,5 +66,5 @@
       <origin xyz="0 0 0" rpy="0 0 0" />
       <geometry>
-        <mesh filename="package://agv_sim/meshes/STEERING_PART_RE2.stl"/>
+        <mesh filename="package://agv_sim/meshes/STEERING_PART_RE2.stl" scale = "0.001 0.001 0.001"/>
       </geometry>
       <material name="white" />
@@ -72,5 +73,5 @@
       <origin xyz="0 0 0" rpy="0 0 0" />
       <geometry>
-        <mesh filename="package://agv_sim/meshes/STEERING_PART_RE2.stl"/>
+        <mesh filename="package://agv_sim/meshes/STEERING_PART_RE2.stl" scale = "0.001 0.001 0.001"/>
       </geometry>
     </collision>
@@ -79,5 +80,6 @@
     <parent link="steering_part" />
     <child link="drive_wheel" />
-    <origin xyz="0.063 0.012 -0.285" rpy="0 0 0" />
+    <!-- <origin xyz="0.063 0.012 -0.285" rpy="0 0 0" /> -->
+    <origin xyz="0.01 0.0 -0.285" rpy="0 0 0" />
     <axis xyz="1 0 0"/>
   </joint>
@@ -156,5 +158,16 @@
     <origin xyz="-0.341 0.103 0.763" rpy="0 0 0"/>
   </joint>
-  <link name="imu_link"/>
+  <link name="imu_link">
+    <!-- <inertial>
+      <mass value="0.641"/>
+      <inertia ixx="0.001" ixy="0.0" ixz="0.0" iyy="0.001" iyz="0.0" izz="0.002"/>
+    </inertial>
+    <visual>
+      <origin xyz="0 0 0" rpy="0 0 0" />
+      <geometry>
+        <mesh filename="package://agv_sim/meshes/IMU.stl" scale = "0.001 0.001 0.001"/>
+      </geometry>
+    </visual> -->
+  </link>
   <joint name="slam_lidar_joint" type="fixed">
     <parent link="base_link" />
@@ -174,5 +187,5 @@
     </visual>
   </link>
-  <joint name="safety_lidar_l_joint" type="fixed">
+  <!-- <joint name="safety_lidar_l_joint" type="fixed">
     <parent link="base_link" />
     <child link="safety_lidar_l" />
@@ -224,4 +237,4 @@
       </geometry>
     </visual>
-  </link>
+  </link> -->
 </robot>

Commit message: agv용 msg추가 - mast_vel만 우선 추가함 - 작업용 메시지 - drive_plugin에 해당 메시지 적용 및 수신 확인

File: agv_sim/urdf/modified_agv.urdf.xacro (robot description, xacro)
@@ -9,6 +9,6 @@
   <link name="base_link">
     <inertial>
-      <origin xyz="0 0 0.89" rpy="0 0 0"/>
-      <mass value="2129.355" />
+      <origin xyz="0 0 0.89" rpy="0 0 0" />
+      <mass value="2522.3" />
       <inertia ixx="990" ixy="0" ixz="0" iyy="990" iyz="0" izz="990" />
     </inertial>
@@ -16,5 +16,5 @@
       <origin xyz="0 0 0" rpy="0 0 1.574" />
       <geometry>
-        <mesh filename="package://agv_sim/meshes/BODY.stl" />
+        <mesh filename="package://agv_sim/meshes/BODY_N_MAST.stl" scale="0.001 0.001 0.001" />
       </geometry>
       <material name="orange" />
@@ -23,17 +23,19 @@
       <origin xyz="0 0 0" rpy="0 0 1.574" />
       <geometry>
-        <mesh filename="package://agv_sim/meshes/BODY.stl"  />
-      </geometry>
-    </collision>
-  </link>
-  <!-- <joint name="mast_joint" type="fixed">
-    <parent link="base_link" />
-    <child link="mast" />
-    <origin xyz="0 0.631 1.875" rpy="0 0 0" />
-  </joint>
-  <link name="mast">
-    <inertial>
-      <mass value="590.628"/>
-      <inertia ixx="1122.228" ixy="-0.195" ixz="1.265" iyy="1071.349" iyz="-243.104" izz="135.921"/>
+        <mesh filename="package://agv_sim/meshes/BODY_N_MAST.stl" scale="0.001 0.001 0.001" />
+      </geometry>
+    </collision>
+  </link>
+  <joint name="fork_joint" type="prismatic">
+    <parent link="base_link" />
+    <child link="fork_house" />
+    <axis xyz="0 0 1"/>
+    <limit lower="2.05" upper="3.07" effort="1000.0" velocity="0.1"/>
+    <origin xyz="-0.631 0 2.07" rpy="0 0 1.574" />
+  </joint>
+  <link name="fork_house">
+    <inertial>
+      <mass value="203.9"/>
+      <inertia ixx="320.5" ixy="0" ixz="0" iyy="34.5" iyz="0" izz="320.5"/>
     </inertial>
     <visual>
@@ -50,21 +52,21 @@
       </geometry>
     </collision>
-  </link> -->
+  </link>
   <joint name="steering_joint" type="continuous">
     <parent link="base_link" />
     <child link="steering_part" />
-    <origin xyz="0.216 0 0.344" rpy="0 0 1.574" />
+    <origin xyz="0.216 0 0.334" rpy="0 0 1.574" />
     <!-- 0.212 -0.0476 0.344 -->
-    <axis xyz="0 0 1"/>
+    <axis xyz="0 0 1" />
   </joint>
   <link name="steering_part">
     <inertial>
-      <mass value="85.056"/>
-      <inertia ixx="2.81" ixy="0.0" ixz="-0.11" iyy="2.77" iyz="0.12" izz="0.9"/>
-    </inertial>
-    <visual>
-      <origin xyz="0 0 0" rpy="0 0 0" />
-      <geometry>
-        <mesh filename="package://agv_sim/meshes/STEERING_PART_RE2.stl" scale = "0.001 0.001 0.001"/>
+      <mass value="85.056" />
+      <inertia ixx="2.81" ixy="0.0" ixz="-0.11" iyy="2.77" iyz="0.12" izz="0.9" />
+    </inertial>
+    <visual>
+      <origin xyz="0 0 0" rpy="0 0 0" />
+      <geometry>
+        <mesh filename="package://agv_sim/meshes/STEERING_PART_RE2.stl" scale="0.001 0.001 0.001" />
       </geometry>
       <material name="white" />
@@ -73,5 +75,5 @@
       <origin xyz="0 0 0" rpy="0 0 0" />
       <geometry>
-        <mesh filename="package://agv_sim/meshes/STEERING_PART_RE2.stl" scale = "0.001 0.001 0.001"/>
+        <mesh filename="package://agv_sim/meshes/STEERING_PART_RE2.stl" scale="0.001 0.001 0.001" />
       </geometry>
     </collision>
@@ -82,15 +84,15 @@
     <!-- <origin xyz="0.063 0.012 -0.285" rpy="0 0 0" /> -->
     <origin xyz="0.01 0.0 -0.285" rpy="0 0 0" />
-    <axis xyz="1 0 0"/>
+    <axis xyz="1 0 0" />
   </joint>
   <link name="drive_wheel">
     <inertial>
-      <mass value="21.755"/>
-      <inertia ixx="0.166" ixy="0.0" ixz="0.0" iyy="0.166" iyz="0.0" izz="0.166"/>
-    </inertial>
-    <visual>
-      <origin xyz="0 0 0" rpy="0 0 0" />
-      <geometry>
-        <mesh filename="package://agv_sim/meshes/DRIVE_WHEEL_RE2.stl"/>
+      <mass value="21.755" />
+      <inertia ixx="0.166" ixy="0.0" ixz="0.0" iyy="0.166" iyz="0.0" izz="0.166" />
+    </inertial>
+    <visual>
+      <origin xyz="0 0 0" rpy="0 0 0" />
+      <geometry>
+        <mesh filename="package://agv_sim/meshes/DRIVE_WHEEL_RE2.stl" />
       </geometry>
       <material name="blue" />
@@ -99,5 +101,5 @@
       <origin xyz="0 0 0" rpy="0 0 0" />
       <geometry>
-        <mesh filename="package://agv_sim/meshes/DRIVE_WHEEL_RE2.stl"/>
+        <mesh filename="package://agv_sim/meshes/DRIVE_WHEEL_RE2.stl" />
       </geometry>
     </collision>
@@ -107,15 +109,15 @@
     <child link="front_wheel_l" />
     <origin xyz="-0.86 -0.451 0.025" rpy="0 0 0" />
-    <axis xyz="0 1 0"/>
+    <axis xyz="0 1 0" />
   </joint>
   <link name="front_wheel_l">
     <inertial>
-      <mass value="16.096"/>
-      <inertia ixx="0.066" ixy="0.0" ixz="0.0" iyy="0.066" iyz="0.0" izz="0.066"/>
-    </inertial>
-    <visual>
-      <origin xyz="0 0 0" rpy="0 0 0" />
-      <geometry>
-        <mesh filename="package://agv_sim/meshes/FRONT_WHEEL_RE2.stl"/>
+      <mass value="16.096" />
+      <inertia ixx="0.066" ixy="0.0" ixz="0.0" iyy="0.066" iyz="0.0" izz="0.066" />
+    </inertial>
+    <visual>
+      <origin xyz="0 0 0" rpy="0 0 0" />
+      <geometry>
+        <mesh filename="package://agv_sim/meshes/FRONT_WHEEL_RE2.stl" />
       </geometry>
       <material name="green" />
@@ -124,5 +126,5 @@
       <origin xyz="0 0 0" rpy="0 0 0" />
       <geometry>
-        <mesh filename="package://agv_sim/meshes/FRONT_WHEEL_RE2.stl"/>
+        <mesh filename="package://agv_sim/meshes/FRONT_WHEEL_RE2.stl" />
       </geometry>
     </collision>
@@ -132,15 +134,15 @@
     <child link="front_wheel_r" />
     <origin xyz="-0.86 0.451 0.025" rpy="0 0 3.14" />
-    <axis xyz="0 1 0"/>
+    <axis xyz="0 1 0" />
   </joint>
   <link name="front_wheel_r">
     <inertial>
-      <mass value="16.096"/>
-      <inertia ixx="0.066" ixy="0.0" ixz="0.0" iyy="0.066" iyz="0.0" izz="0.066"/>
-    </inertial>
-    <visual>
-      <origin xyz="0 0 0" rpy="0 0 0" />
-      <geometry>
-        <mesh filename="package://agv_sim/meshes/FRONT_WHEEL_RE2.stl"/>
+      <mass value="16.096" />
+      <inertia ixx="0.066" ixy="0.0" ixz="0.0" iyy="0.066" iyz="0.0" izz="0.066" />
+    </inertial>
+    <visual>
+      <origin xyz="0 0 0" rpy="0 0 0" />
+      <geometry>
+        <mesh filename="package://agv_sim/meshes/FRONT_WHEEL_RE2.stl" />
       </geometry>
       <material name="green" />
@@ -149,12 +151,12 @@
       <origin xyz="0 0 0" rpy="0 0 0" />
       <geometry>
-        <mesh filename="package://agv_sim/meshes/FRONT_WHEEL_RE2.stl"/>
+        <mesh filename="package://agv_sim/meshes/FRONT_WHEEL_RE2.stl" />
       </geometry>
     </collision>
   </link>
   <joint name="imu_joint" type="fixed">
-    <parent link="base_link"/>
-    <child link="imu_link"/>
-    <origin xyz="-0.341 0.103 0.763" rpy="0 0 0"/>
+    <parent link="base_link" />
+    <child link="imu_link" />
+    <origin xyz="-0.341 0.103 0.763" rpy="0 0 0" />
   </joint>
   <link name="imu_link">
@@ -177,11 +179,11 @@
   <link name="slam_lidar">
     <inertial>
-      <mass value="0.641"/>
-      <inertia ixx="0.001" ixy="0.0" ixz="0.0" iyy="0.001" iyz="0.0" izz="0.002"/>
-    </inertial>
-    <visual>
-      <origin xyz="0 0 0" rpy="0 0 0" />
-      <geometry>
-        <mesh filename="package://agv_sim/meshes/C16_3D.stl" scale = "0.001 0.001 0.001"/>
+      <mass value="0.641" />
+      <inertia ixx="0.001" ixy="0.0" ixz="0.0" iyy="0.001" iyz="0.0" izz="0.002" />
+    </inertial>
+    <visual>
+      <origin xyz="0 0 0" rpy="0 0 0" />
+      <geometry>
+        <mesh filename="package://agv_sim/meshes/C16_3D.stl" scale="0.001 0.001 0.001" />
       </geometry>
     </visual>

Commit message: 시뮬레이션에서 Fork_House 움직임 구현

File: agv_sim/urdf/modified_agv.urdf.xacro (robot description, xacro)
@@ -31,16 +31,17 @@
     <child link="fork_house" />
     <axis xyz="0 0 1"/>
-    <limit lower="2.05" upper="3.07" effort="1000.0" velocity="0.1"/>
-    <origin xyz="-0.631 0 2.07" rpy="0 0 1.574" />
+    <limit lower="-0.05" upper="1.5" effort="1000.0" velocity="0.1"/>
+    <origin xyz="-0.989 0 0.1" rpy="0 0 1.574" />
   </joint>
   <link name="fork_house">
     <inertial>
-      <mass value="203.9"/>
-      <inertia ixx="320.5" ixy="0" ixz="0" iyy="34.5" iyz="0" izz="320.5"/>
-    </inertial>
-    <visual>
-      <origin xyz="0 0 0" rpy="0 0 0" />
-      <geometry>
-        <mesh filename="package://agv_sim/meshes/MAST.stl" scale = "0.001 0.001 0.001" />
+      <mass value="0.1"/>
+      <inertia ixx="0.0" ixy="0.0" ixz="0.0" iyy="0.0" iyz="0.0" izz="0.0"/>
+      <!-- <inertia ixx="320.5" ixy="0" ixz="0" iyy="34.5" iyz="0" izz="320.5"/> -->
+    </inertial>
+    <visual>
+      <origin xyz="0 0 0" rpy="0 0 0" />
+      <geometry>
+        <mesh filename="package://agv_sim/meshes/FORK_HOUSE_RE.stl" scale = "0.001 0.001 0.001" />
       </geometry>
       <material name="dark_grey" />
@@ -49,5 +50,5 @@
       <origin xyz="0 0 0" rpy="0 0 0" />
       <geometry>
-        <mesh filename="package://agv_sim/meshes/MAST.stl" scale = "0.001 0.001 0.001" />
+        <mesh filename="package://agv_sim/meshes/FORK_HOUSE_RE.stl" scale = "0.001 0.001 0.001" />
       </geometry>
     </collision>

Commit message: SLAM시 Odometry 변경  - 드라이브 플러그인의 오도메트리 계산 제거  - cartographer에서 제공하는 LiDAR 및 IMU를 이용한 Odometry 사용

File: agv_sim/urdf/modified_agv.urdf.xacro (robot description, xacro)
@@ -31,5 +31,5 @@
     <child link="fork_house" />
     <axis xyz="0 0 1"/>
-    <limit lower="-0.05" upper="1.5" effort="1000.0" velocity="0.1"/>
+    <limit lower="-0.11" upper="1.5" effort="1000.0" velocity="0.1"/>
     <origin xyz="-0.989 0 0.1" rpy="0 0 1.574" />
   </joint>
