Commit message: 모델파일 일부 수정 및 드라이브 플러그인에서 odom발행으로 다시 재 수정

File: agv_sim/urdf/final_agv.urdf.xacro (robot description, xacro)
@@ -5,9 +5,9 @@
     <parent link="base_footprint" />
     <child link="base_link" />
-    <origin xyz="0 0 0.1" rpy="0 0 0" />
+    <origin xyz="0 0 0.18" rpy="0 0 0" />
   </joint>
   <link name="base_link">
     <inertial>
-      <origin xyz="0 0 0.89" rpy="0 0 0" />
+      <origin xyz="0 0 0.81" rpy="0 0 0" />
       <mass value="2522.3" />
       <inertia ixx="990" ixy="0" ixz="0" iyy="990" iyz="0" izz="990" />
@@ -32,5 +32,5 @@
     <axis xyz="0 0 1"/>
     <limit lower="-0.11" upper="1.5" effort="1000.0" velocity="0.1"/>
-    <origin xyz="-0.989 0 0.1" rpy="0 0 1.574" />
+    <origin xyz="-0.989 0 0.18" rpy="0 0 1.574" />
   </joint>
   <link name="fork_house">
@@ -38,5 +38,4 @@
       <mass value="0.1"/>
       <inertia ixx="0.0" ixy="0.0" ixz="0.0" iyy="0.0" iyz="0.0" izz="0.0"/>
-      <!-- <inertia ixx="320.5" ixy="0" ixz="0" iyy="34.5" iyz="0" izz="320.5"/> -->
     </inertial>
     <visual>
@@ -54,9 +53,9 @@
     </collision>
   </link>
+  <!-- <joint name="steering_joint" type="fixed"> -->
   <joint name="steering_joint" type="continuous">
     <parent link="base_link" />
     <child link="steering_part" />
-    <origin xyz="0.216 0 0.334" rpy="0 0 1.574" />
-    <!-- 0.212 -0.0476 0.344 -->
+    <origin xyz="0.216 0 0.414" rpy="0 0 1.574" />
     <axis xyz="0 0 1" />
   </joint>
@@ -80,8 +79,8 @@
     </collision>
   </link>
+  <!-- <joint name="drive_wheel_joint" type="fixed"> -->
   <joint name="drive_wheel_joint" type="continuous">
     <parent link="steering_part" />
     <child link="drive_wheel" />
-    <!-- <origin xyz="0.063 0.012 -0.285" rpy="0 0 0" /> -->
     <origin xyz="0.01 0.0 -0.285" rpy="0 0 0" />
     <axis xyz="1 0 0" />
@@ -109,5 +108,5 @@
     <parent link="base_link" />
     <child link="front_wheel_l" />
-    <origin xyz="-0.86 -0.451 0.025" rpy="0 0 0" />
+    <origin xyz="-0.86 -0.451 0.105" rpy="0 0 0" />
     <axis xyz="0 1 0" />
   </joint>
@@ -134,5 +133,5 @@
     <parent link="base_link" />
     <child link="front_wheel_r" />
-    <origin xyz="-0.86 0.451 0.025" rpy="0 0 3.14" />
+    <origin xyz="-0.86 0.451 0.105" rpy="0 0 3.14" />
     <axis xyz="0 1 0" />
   </joint>
@@ -159,22 +158,11 @@
     <parent link="base_link" />
     <child link="imu_link" />
-    <origin xyz="-0.341 0.103 0.763" rpy="0 0 0" />
-  </joint>
-  <link name="imu_link">
-    <!-- <inertial>
-      <mass value="0.641"/>
-      <inertia ixx="0.001" ixy="0.0" ixz="0.0" iyy="0.001" iyz="0.0" izz="0.002"/>
-    </inertial>
-    <visual>
-      <origin xyz="0 0 0" rpy="0 0 0" />
-      <geometry>
-        <mesh filename="package://agv_sim/meshes/IMU.stl" scale = "0.001 0.001 0.001"/>
-      </geometry>
-    </visual> -->
-  </link>
+    <origin xyz="-0.341 0.103 0.843" rpy="0 0 0" />
+  </joint>
+  <link name="imu_link" />
   <joint name="slam_lidar_joint" type="fixed">
     <parent link="base_link" />
     <child link="slam_lidar" />
-    <origin xyz="0 -0.2 2.197" rpy="0 0 0" />
+    <origin xyz="0 -0.2 2.277" rpy="0 0 0" />
   </joint>
   <link name="slam_lidar">
@@ -197,11 +185,11 @@
   <link name="safety_lidar_l">
     <inertial>
-      <mass value="0.295"/>
-      <inertia ixx="0.001" ixy="0.0" ixz="0.0" iyy="0.001" iyz="0.0" izz="0.002"/>
+      <mass value="0.295" />
+      <inertia ixx="0.001" ixy="0.0" ixz="0.0" iyy="0.001" iyz="0.0" izz="0.002" />
     </inertial>
     <visual>
       <origin xyz="0 0 0" rpy="-1.57 0 1.57" />
       <geometry>
-        <mesh filename="package://agv_sim/meshes/2D_SAFETY_LIDAR.stl" scale = "0.001 0.001 0.001"/>
+        <mesh filename="package://agv_sim/meshes/2D_SAFETY_LIDAR.stl" scale="0.001 0.001 0.001" />
       </geometry>
     </visual>
@@ -214,11 +202,11 @@
   <link name="safety_lidar_r">
     <inertial>
-      <mass value="0.295"/>
-      <inertia ixx="0.001" ixy="0.0" ixz="0.0" iyy="0.001" iyz="0.0" izz="0.002"/>
+      <mass value="0.295" />
+      <inertia ixx="0.001" ixy="0.0" ixz="0.0" iyy="0.001" iyz="0.0" izz="0.002" />
     </inertial>
     <visual>
       <origin xyz="0 0 0" rpy="-1.57 0 1.56" />
       <geometry>
-        <mesh filename="package://agv_sim/meshes/2D_SAFETY_LIDAR.stl" scale = "0.001 0.001 0.001"/>
+        <mesh filename="package://agv_sim/meshes/2D_SAFETY_LIDAR.stl" scale="0.001 0.001 0.001" />
       </geometry>
     </visual>
@@ -231,11 +219,11 @@
   <link name="safety_lidar_m">
     <inertial>
-      <mass value="0.295"/>
-      <inertia ixx="0.001" ixy="0.0" ixz="0.0" iyy="0.001" iyz="0.0" izz="0.002"/>
+      <mass value="0.295" />
+      <inertia ixx="0.001" ixy="0.0" ixz="0.0" iyy="0.001" iyz="0.0" izz="0.002" />
     </inertial>
     <visual>
       <origin xyz="0 0 0" rpy="-1.57 0 1.57" />
       <geometry>
-        <mesh filename="package://agv_sim/meshes/2D_SAFETY_LIDAR.stl" scale = "0.001 0.001 0.001"/>
+        <mesh filename="package://agv_sim/meshes/2D_SAFETY_LIDAR.stl" scale="0.001 0.001 0.001" />
       </geometry>
     </visual>

File: agv_sim/urdf/modified_agv_description.urdf.xacro (robot description, xacro)
@@ -18,5 +18,5 @@
   </material>
   <!-- this include provides the macro definition used below -->
- <xacro:include filename="$(find agv_sim)/urdf/modified_agv.urdf.xacro"/>
+ <xacro:include filename="$(find agv_sim)/urdf/final_agv.urdf.xacro"/>
  <xacro:property name="model" value="(arg model)"/>
  <!-- if more models are defined, add them here -->

Commit message: 로컬 플래너 수정 중 - 회전 반경 - 회전 속도 등 - dwb => RegulatedPurePursuit

File: agv_sim/urdf/final_agv.urdf.xacro (robot description, xacro)
@@ -158,5 +158,5 @@
     <parent link="base_link" />
     <child link="imu_link" />
-    <origin xyz="-0.341 0.103 0.843" rpy="0 0 0" />
+    <origin xyz="0 0 0" rpy="0 0 0" />
   </joint>
   <link name="imu_link" />

Commit message: nav2에서 회전을 제대로 컨트롤하기가 힘듦 해결책으로 일정 지점 목적지로 정해 질 경우 행동을 시나리오화 하고 이를 실행 할 시나리오 작성 중

File: agv_sim/urdf/final_agv.urdf.xacro (robot description, xacro)
@@ -164,5 +164,5 @@
     <parent link="base_link" />
     <child link="slam_lidar" />
-    <origin xyz="0 -0.2 2.277" rpy="0 0 0" />
+    <origin xyz="0.2 0 2.277" rpy="0 0 0" />
   </joint>
   <link name="slam_lidar">

Commit message: 자율주행 시 로봇 중심점 변경 sim_time을 사용하도록 변경 드라이브 플러그인 일부 변경

File: agv_sim/urdf/final_agv.urdf.xacro (robot description, xacro)
@@ -5,5 +5,5 @@
     <parent link="base_footprint" />
     <child link="base_link" />
-    <origin xyz="0 0 0.18" rpy="0 0 0" />
+    <origin xyz="0.7 0 0.18" rpy="0 0 0" />
   </joint>
   <link name="base_link">
@@ -53,5 +53,4 @@
     </collision>
   </link>
-  <!-- <joint name="steering_joint" type="fixed"> -->
   <joint name="steering_joint" type="continuous">
     <parent link="base_link" />
@@ -79,5 +78,4 @@
     </collision>
   </link>
-  <!-- <joint name="drive_wheel_joint" type="fixed"> -->
   <joint name="drive_wheel_joint" type="continuous">
     <parent link="steering_part" />

Commit message: 접촉센서 추가 및 접촉 시 정지 추가

File: agv_sim/urdf/final_agv.urdf.xacro (robot description, xacro)
@@ -227,3 +227,49 @@
     </visual>
   </link>
+  <joint name="bumper_r_joint" type="fixed">
+    <parent link="base_link" />
+    <child link="bumper_r_link" />
+    <origin xyz="-1.09 0.193 0.35" rpy="0 0 0" />
+  </joint>
+  <link name="bumper_r_link">
+    <inertial>
+      <mass value="0.295" />
+      <inertia ixx="0.001" ixy="0.0" ixz="0.0" iyy="0.001" iyz="0.0" izz="0.002" />
+    </inertial>
+    <visual>
+      <origin xyz="0 0 0" rpy="0 0 0" />
+      <geometry>
+        <box size="0.01 0.04 0.12"/>
+      </geometry>
+    </visual>
+    <collision>
+      <origin xyz="0 0 0" rpy="0 0 0" />
+      <geometry>
+        <box size="0.01 0.04 0.12"/>
+      </geometry>
+    </collision>
+  </link>
+  <joint name="bumper_l_joint" type="fixed">
+    <parent link="base_link" />
+    <child link="bumper_l_link" />
+    <origin xyz="-1.09 -0.193 0.35" rpy="0 0 0" />
+  </joint>
+  <link name="bumper_l_link">
+    <inertial>
+      <mass value="0.295" />
+      <inertia ixx="0.001" ixy="0.0" ixz="0.0" iyy="0.001" iyz="0.0" izz="0.002" />
+    </inertial>
+    <visual>
+      <origin xyz="0 0 0" rpy="0 0 0" />
+      <geometry>
+        <box size="0.01 0.04 0.12"/>
+      </geometry>
+    </visual>
+    <collision>
+      <origin xyz="0 0 0" rpy="0 0 0" />
+      <geometry>
+        <box size="0.01 0.04 0.12"/>
+      </geometry>
+    </collision>
+  </link>
 </robot>

Commit message: rs232 update motor control 추가 odometry 및 joint_state 추가

File: agv_sim/urdf/final_agv.urdf.xacro (robot description, xacro)
@@ -162,5 +162,5 @@
     <parent link="base_link" />
     <child link="slam_lidar" />
-    <origin xyz="0.2 0 2.277" rpy="0 0 0" />
+    <origin xyz="0.2 0 2.277" rpy="0 0 0.785" />
   </joint>
   <link name="slam_lidar">

Commit message: agv_com pkg   - rs232 imu to pc   - can_bus imu   - 단위 변경 및 적용     -> G to m/s^2     -> dps to rad/s To Do   - Check TF     - 슬램 실행 시 뒤집혀서 나옴

File: agv_sim/urdf/final_agv.urdf.xacro (robot description, xacro)
@@ -156,5 +156,6 @@
     <parent link="base_link" />
     <child link="imu_link" />
-    <origin xyz="0 0 0" rpy="0 0 0" />
+    <!-- <origin 0.216 xyz="0.7 0 0.18" rpy="0 0 0" /> -->
+    <origin xyz="-0.5 0 0.82" rpy="0 0 0" />
   </joint>
   <link name="imu_link" />
@@ -162,5 +163,5 @@
     <parent link="base_link" />
     <child link="slam_lidar" />
-    <origin xyz="0.2 0 2.277" rpy="0 0 0.785" />
+    <origin xyz="0.2 0 2.277" rpy="0 0 1.57" />
   </joint>
   <link name="slam_lidar">
@@ -227,5 +228,5 @@
     </visual>
   </link>
-  <joint name="bumper_r_joint" type="fixed">
+  <!-- <joint name="bumper_r_joint" type="fixed">
     <parent link="base_link" />
     <child link="bumper_r_link" />
@@ -272,4 +273,4 @@
       </geometry>
     </collision>
-  </link>
+  </link> -->
 </robot>
